Commit message: Fixed PushCorp tool orientation

File: src/khi_cx_description/urdf/cx165l_macro.xacro (robot description, xacro)
@@ -292,5 +292,5 @@
     <!-- PushCorp Compliant Tool and Spindle -->
     <joint name="${prefix}pushcorp" type="fixed">
-      <origin xyz="0 0.0949325000000025 0" rpy="0 1.5707963267949 0" />
+      <origin xyz="0 0.094933 0" rpy="0 1.5708 0" />
       <parent link="${prefix}link6"/>
       <child link="${prefix}pushcorp"/>

Commit message: Restructured urdf to workcell.xacro format

File: src/khi_cx_description/urdf/cx165l_macro.xacro (robot description, xacro)
@@ -4,5 +4,4 @@
     <xacro:include filename="$(find khi_cx_description)/urdf/cx.transmission.xacro" />
     <xacro:include filename="$(find khi_cx_description)/urdf/common.gazebo.xacro" />
-    <xacro:include filename="$(find khi_cx_description)/urdf/isu_lab.xacro" />
     <!-- link rviz colors -->
     <material name="White">
@@ -290,36 +289,4 @@
         <xacro:default_inertial mass="${j6_mass}"/>
     </link>
-    <!-- PushCorp Compliant Tool and Spindle -->
-    <joint name="${prefix}pushcorp" type="fixed">
-      <origin xyz="0 0.094933 0" rpy="0 1.5708 0" />
-      <parent link="${prefix}link6"/>
-      <child link="${prefix}pushcorp"/>
-    </joint>
-    <link name="${prefix}pushcorp">
-        <visual>
-            <origin
-                xyz="0 0 0"
-                rpy="0 0 0" />
-            <geometry>
-                <mesh
-                filename="package://khi_cx_description/meshes/CX165L-PUSHCORP.STL" />
-            </geometry>
-            <material
-                name="">
-                <color
-                rgba="0.75294 0.75294 0.75294 1" />
-            </material>
-        </visual>
-        <collision>
-            <origin
-                xyz="0 0 0"
-                rpy="0 0 0" />
-            <geometry>
-                <mesh
-                filename="package://khi_cx_description/meshes/CX165L-PUSHCORP-HULL.STL" />
-            </geometry>
-        </collision>
-        <xacro:default_inertial mass="${j6_mass}"/>
-    </link>
   </xacro:macro>
 </robot>

File: src/khi_cx_description/urdf/isu_lab.xacro (robot description, xacro)
@@ -1,5 +1,4 @@
 <?xml version="1.0"?>
 <robot xmlns:xacro="http://ros.org/wiki/xacro">
-      <!-- link inertial(TODO : set correct link inertial )-->
     <xacro:macro name="default_inertial" params="mass">
       <inertial>
@@ -9,86 +8,4 @@
     </xacro:macro>
     <!-- Lab Environment -->
-     <link name="base_plate">
-        <visual>
-            <origin
-                xyz="0 0 0.0127"
-                rpy="0 0 0" />
-            <geometry>
-                <box size="1.016 1.016 0.0254" />
-            </geometry>
-            <material
-                name="">
-                <color
-                rgba="0.75294 0.75294 0.75294 1" />
-            </material>
-        </visual>
-        <collision>
-            <origin
-                xyz="0 0 0.0127"
-                rpy="0 0 0" />
-            <geometry>
-                <box size="1.016 1.016 0.0254" />
-            </geometry>
-        </collision>
-        <xacro:default_inertial mass="1"/>
-    </link>
-    <joint name="world2east_wall" type="fixed">
-        <parent link="world"/>
-        <child link="east_wall"/>
-        <origin rpy="0 0 0" xyz="0 0 0"/>
-    </joint>
-    <link name="east_wall">
-        <visual>
-            <origin
-                xyz="-0.7888 -0.7612 2.5"
-                rpy="0 0 0" />
-            <geometry>
-                <box size="3 0.1 5" />
-            </geometry>
-            <material
-                name="">
-                <color
-                rgba="0.75294 0.75294 0.75294 1" />
-            </material>
-        </visual>
-        <collision>
-            <origin
-                xyz="-0.7888 -0.7612 2.5"
-                rpy="0 0 0" />
-            <geometry>
-                <box size="3 0.1 5" />
-            </geometry>
-        </collision>
-        <xacro:default_inertial mass="1"/>
-    </link>
-    <joint name="world2north_wall" type="fixed">
-        <parent link="world"/>
-        <child link="north_wall"/>
-        <origin rpy="0 0 0" xyz="0 0 0"/>
-    </joint>
-    <link name="north_wall">
-        <visual>
-            <origin
-                xyz="0.7612 0.9398 2.5"
-                rpy="0 0 0" />
-            <geometry>
-                <box size="0.1 3.302 5" />
-            </geometry>
-            <material
-                name="">
-                <color
-                rgba="0.75294 0.75294 0.75294 1" />
-            </material>
-        </visual>
-        <collision>
-            <origin
-                xyz="0.7612 0.9398 2.5"
-                rpy="0 0 0" />
-            <geometry>
-                <box size="0.1 3.302 5" />
-            </geometry>
-        </collision>
-        <xacro:default_inertial mass="1"/>
-    </link>
     <joint name="world2floor" type="fixed">
         <parent link="world"/>
@@ -120,6 +37,93 @@
         <xacro:default_inertial mass="1"/>
     </link>
-    <joint name="world2westwall" type="fixed">
-        <parent link="world"/>
+    <joint name="floor2base_plate" type="fixed">
+        <parent link="floor"/>
+        <child link="base_plate"/>
+        <origin rpy="0 0 0" xyz="0 0 0"/>
+    </joint>
+     <link name="base_plate">
+        <visual>
+            <origin
+                xyz="0 0 0.0127"
+                rpy="0 0 0" />
+            <geometry>
+                <box size="1.016 1.016 0.0254" />
+            </geometry>
+            <material
+                name="">
+                <color
+                rgba="0.75294 0.75294 0.75294 1" />
+            </material>
+        </visual>
+        <collision>
+            <origin
+                xyz="0 0 0.0127"
+                rpy="0 0 0" />
+            <geometry>
+                <box size="1.016 1.016 0.0254" />
+            </geometry>
+        </collision>
+        <xacro:default_inertial mass="1"/>
+    </link>
+    <joint name="floor2east_wall" type="fixed">
+        <parent link="floor"/>
+        <child link="east_wall"/>
+        <origin rpy="0 0 0" xyz="0 0 0"/>
+    </joint>
+    <link name="east_wall">
+        <visual>
+            <origin
+                xyz="-0.7888 -0.7612 2.5"
+                rpy="0 0 0" />
+            <geometry>
+                <box size="3 0.1 5" />
+            </geometry>
+            <material
+                name="">
+                <color
+                rgba="0.75294 0.75294 0.75294 1" />
+            </material>
+        </visual>
+        <collision>
+            <origin
+                xyz="-0.7888 -0.7612 2.5"
+                rpy="0 0 0" />
+            <geometry>
+                <box size="3 0.1 5" />
+            </geometry>
+        </collision>
+        <xacro:default_inertial mass="1"/>
+    </link>
+    <joint name="floor2north_wall" type="fixed">
+        <parent link="floor"/>
+        <child link="north_wall"/>
+        <origin rpy="0 0 0" xyz="0 0 0"/>
+    </joint>
+    <link name="north_wall">
+        <visual>
+            <origin
+                xyz="0.7612 0.9398 2.5"
+                rpy="0 0 0" />
+            <geometry>
+                <box size="0.1 3.302 5" />
+            </geometry>
+            <material
+                name="">
+                <color
+                rgba="0.75294 0.75294 0.75294 1" />
+            </material>
+        </visual>
+        <collision>
+            <origin
+                xyz="0.7612 0.9398 2.5"
+                rpy="0 0 0" />
+            <geometry>
+                <box size="0.1 3.302 5" />
+            </geometry>
+        </collision>
+        <xacro:default_inertial mass="1"/>
+    </link>
+    <joint name="floor2westwall" type="fixed">
+        <parent link="floor"/>
         <child link="west_wall"/>
         <origin rpy="0 0 0" xyz="0 0 0"/>
@@ -149,6 +153,6 @@
         <xacro:default_inertial mass="1"/>
     </link>
-    <joint name="world2south_wall" type="fixed">
-        <parent link="world"/>
+    <joint name="floor2south_wall" type="fixed">
+        <parent link="floor"/>
         <child link="south_wall"/>
         <origin rpy="0 0 0" xyz="0 0 0"/>

Commit message: New ISU-LAB URDF, real robot connection changes

File: src/khi_cx_description/urdf/cx165l_macro.xacro (robot description, xacro)
@@ -48,5 +48,5 @@
     </xacro:macro>
     <joint name="${prefix}base_link_joint" type="fixed">
-        <parent link="base_plate" />
+        <parent link="world" />
         <child link="base_link" />
         <origin rpy="0 0 0" xyz="0 0 0" />
@@ -116,5 +116,5 @@
     <!-- Link 2 -->
     <joint name="${prefix}joint2" type="revolute">
-      <axis xyz="1 0 0" rpy="0 0 0" />
+      <axis xyz="-1 0 0" rpy="0 0 0" />
       <limit effort="1000.0" lower="${j2_lower_limit}" upper="${j2_upper_limit}" velocity="${j2_velocity_limit}"/>
       <origin xyz="0 0.3 0" rpy="0 0 0" />

File: src/khi_cx_description/urdf/isu_lab.xacro (robot description, xacro)
@@ -8,16 +8,17 @@
     </xacro:macro>
     <!-- Lab Environment -->
-    <joint name="world2floor" type="fixed">
+    <joint name="world2isu_lab" type="fixed">
         <parent link="world"/>
-        <child link="floor"/>
+        <child link="isu_lab"/>
         <origin rpy="0 0 0" xyz="0 0 0"/>
     </joint>
-    <link name="floor">
+    <link name="isu_lab">
         <visual>
             <origin
-                xyz="0 0 -0.05"
+                xyz="0 0 0"
                 rpy="0 0 0" />
             <geometry>
-                <box size="6 6 0.1" />
+                <mesh
+                filename="package://khi_cx_description/meshes/ISU-LAB.STL" />
             </geometry>
             <material
@@ -29,153 +30,9 @@
         <collision>
             <origin
-                xyz="0 0 -0.05"
+                xyz="0 0 0"
                 rpy="0 0 0" />
             <geometry>
-                <box size="6 6 0.1" />
-            </geometry>
-        </collision>
-        <xacro:default_inertial mass="1"/>
-    </link>
-    <joint name="floor2base_plate" type="fixed">
-        <parent link="floor"/>
-        <child link="base_plate"/>
-        <origin rpy="0 0 0" xyz="0 0 0"/>
-    </joint>
-     <link name="base_plate">
-        <visual>
-            <origin
-                xyz="0 0 0.0127"
-                rpy="0 0 0" />
-            <geometry>
-                <box size="1.016 1.016 0.0254" />
-            </geometry>
-            <material
-                name="">
-                <color
-                rgba="0.75294 0.75294 0.75294 1" />
-            </material>
-        </visual>
-        <collision>
-            <origin
-                xyz="0 0 0.0127"
-                rpy="0 0 0" />
-            <geometry>
-                <box size="1.016 1.016 0.0254" />
-            </geometry>
-        </collision>
-        <xacro:default_inertial mass="1"/>
-    </link>
-    <joint name="floor2east_wall" type="fixed">
-        <parent link="floor"/>
-        <child link="east_wall"/>
-        <origin rpy="0 0 0" xyz="0 0 0"/>
-    </joint>
-    <link name="east_wall">
-        <visual>
-            <origin
-                xyz="-0.7888 -0.7612 2.5"
-                rpy="0 0 0" />
-            <geometry>
-                <box size="3 0.1 5" />
-            </geometry>
-            <material
-                name="">
-                <color
-                rgba="0.75294 0.75294 0.75294 1" />
-            </material>
-        </visual>
-        <collision>
-            <origin
-                xyz="-0.7888 -0.7612 2.5"
-                rpy="0 0 0" />
-            <geometry>
-                <box size="3 0.1 5" />
-            </geometry>
-        </collision>
-        <xacro:default_inertial mass="1"/>
-    </link>
-    <joint name="floor2north_wall" type="fixed">
-        <parent link="floor"/>
-        <child link="north_wall"/>
-        <origin rpy="0 0 0" xyz="0 0 0"/>
-    </joint>
-    <link name="north_wall">
-        <visual>
-            <origin
-                xyz="0.7612 0.9398 2.5"
-                rpy="0 0 0" />
-            <geometry>
-                <box size="0.1 3.302 5" />
-            </geometry>
-            <material
-                name="">
-                <color
-                rgba="0.75294 0.75294 0.75294 1" />
-            </material>
-        </visual>
-        <collision>
-            <origin
-                xyz="0.7612 0.9398 2.5"
-                rpy="0 0 0" />
-            <geometry>
-                <box size="0.1 3.302 5" />
-            </geometry>
-        </collision>
-        <xacro:default_inertial mass="1"/>
-    </link>
-    <joint name="floor2westwall" type="fixed">
-        <parent link="floor"/>
-        <child link="west_wall"/>
-        <origin rpy="0 0 0" xyz="0 0 0"/>
-    </joint>
-    <link name="west_wall">
-        <visual>
-            <origin
-                xyz="-0.7888 2.6392 2.5"
-                rpy="0 0 0" />
-            <geometry>
-                <box size="3 0.1 5" />
-            </geometry>
-            <material
-                name="">
-                <color
-                rgba="0.75294 0.75294 0.75294 0.2" />
-            </material>
-        </visual>
-        <collision>
-            <origin
-                xyz="-0.7888 2.6392 2.5"
-                rpy="0 0 0" />
-            <geometry>
-                <box size="3 0.1 5" />
-            </geometry>
-        </collision>
-        <xacro:default_inertial mass="1"/>
-    </link>
-    <joint name="floor2south_wall" type="fixed">
-        <parent link="floor"/>
-        <child link="south_wall"/>
-        <origin rpy="0 0 0" xyz="0 0 0"/>
-    </joint>
-    <link name="south_wall">
-        <visual>
-            <origin
-                xyz="-2.3344 0.9398 2.5"
-                rpy="0 0 0" />
-            <geometry>
-                <box size="0.1 3.302 5" />
-            </geometry>
-            <material
-                name="">
-                <color
-                rgba="0.75294 0.75294 0.75294 0.2" />
-            </material>
-        </visual>
-        <collision>
-            <origin
-                xyz="-2.3344 0.9398 2.5"
-                rpy="0 0 0" />
-            <geometry>
-                <box size="0.1 3.302 5" />
+                <mesh
+                filename="package://khi_cx_description/meshes/ISU-LAB.STL" />
             </geometry>
         </collision>
